File: Board/Capacitive Moisture Sensor REV 02.sch (EAGLE design)
At the start: 19 parts, among them U1 TLC555CP, U2 LM358N, X1 22-23-2041

Commit message: Completed board layout for rework modification
Parts:
- added R10, R8: 1M, rcl:R-US_R1206
- C3: value 100pF -> 10nF
- R1: value 4.7k -> 3.3k
- R2: value 680 -> 3.3k
- R3: value 1k -> 10k
- R4: value 5.1k -> 750k
- R9: value 1k -> 3.3k
Connections:
- new net N$1: U2B.-IN, U2B.OUT
- new net N$11: R10.2, R8.1, U2B.+IN
- net +5V: now also R10.1
- net GND: now also R8.2; no longer U2B.+IN, U2B.-IN, U2B.OUT
Other:
- note added: "6.67kHz Square Wave 60us HIGH 90us LOW"
- note added: "Unused amplication pin"
- note removed: "959.7 Hz Square Wave 501ms HIGH 541 ms LOW"
- moved on the sheet: U2B

Commit message: Updated text in schematic
Other:
- note added: "6.4kHz PWM Nominally 81.0us HIGH Nominally 75.2us LOW Nominally"
- note added: "Unused OP-Amp pins"
- note removed: "6.67kHz Square Wave 60us HIGH 90us LOW"
- note removed: "Unused amplication pin"
Changed lines of the file:
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@@
 <?xml version="1.0" encoding="utf-8"?>
 <!DOCTYPE eagle SYSTEM "eagle.dtd">
-<eagle version="9.6.1">
+<eagle version="9.6.2">
 <drawing>
 <settings>
@@
 <plain>
 <text x="-50.8" y="157.48" size="2.54" layer="97">Buffer (Voltage Follower)</text>
-<text x="-218.44" y="162.56" size="3.81" layer="97">6.67kHz Square Wave
-60us  HIGH
-90us LOW </text>
+<text x="-218.44" y="170.18" size="3.302" layer="97">6.4kHz  PWM Nominally
+81.0us  HIGH Nominally
+75.2us  LOW Nominally</text>
 <wire x1="-114.3" y1="185.42" x2="-114.3" y2="83.82" width="0.1524" layer="97" style="shortdash"/>
 <wire x1="-114.3" y1="83.82" x2="-220.98" y2="83.82" width="0.1524" layer="97" style="shortdash"/>
@@
 C = Ks * 5.208pF
 Ks (Solder mask Dielectric constant) = 3.8</text>
-<text x="-33.02" y="101.6" size="2.54" layer="97">Unused amplication pin</text>
+<text x="-33.02" y="101.6" size="2.54" layer="97">Unused OP-Amp pins</text>
 </plain>
 <instances>
